File: Assets/PCB/flatFoot.kicad_pcb (KiCad board)
At the start: 2 copper layers, 124.5 x 63.5 mm, 17 parts

Commit message: Update flatFoot.kicad_pcb
Parts:
- added REF**: PinHeader_1x02_P2.54mm_Vertical, Connector_PinHeader_2.54mm:PinHeader_1x02_P2.54mm_Vertical, F.Cu at (194.1, 87.9)
Routing:
- net (no net): track 1645.3 -> 1899.8 mm, vias 48 -> 53
Other:
- outline, holes or cut-outs redrawn
