File: Assets/PCB/circle.kicad_pcb (KiCad board)
At the start: 2 copper layers, 40.6 x 40.6 mm, 21 parts, among them j1 R_0805_2012Metric, j10 R_0805_2012Metric, j11 R_0805_2012Metric, j12 R_0805_2012Metric, j13 R_0805_2012Metric, j14 R_0805_2012Metric, j15 R_0805_2012Metric, j2 R_0805_2012Metric, j3 R_0805_2012Metric, j4 R_0805_2012Metric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

Commit message: fixed PCBs
Changed lines of the file:
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@@
   (gr_line (start 118.364 106.426) (end 122.682 106.426)
     (stroke (width 0.2) (type default)) (layer "F.Cu"))
+  (gr_line (start 125.73 97.282) (end 124.206 97.282)
+    (stroke (width 0.2) (type default)) (layer "F.Cu"))
   (gr_line (start 116.332 90.932) (end 116.332 88.138)
     (stroke (width 0.2) (type default)) (layer "F.Cu"))
@@
   (gr_line (start 118.364 112.522) (end 118.364 106.426)
     (stroke (width 0.2) (type default)) (layer "F.Cu"))
+  (gr_line (start 125.73 98.552) (end 123.444 98.552)
+    (stroke (width 0.2) (type default)) (layer "F.Cu"))
   (gr_line (start 124.714 115.316) (end 125.73 115.316)
     (stroke (width 0.2) (type default)) (layer "F.Cu"))
@@
   (gr_line (start 119.38 97.282) (end 119.681 98.552)
     (stroke (width 0.2) (type default)) (layer "F.Cu"))
+  (gr_line (start 125.984 96.012) (end 124.206 96.012)
+    (stroke (width 0.2) (type default)) (layer "F.Cu"))
   (gr_line (start 123.698 96.012) (end 123.698 95.25)
     (stroke (width 0.2) (type default)) (layer "F.Cu"))
@@
   (gr_line (start 122.174 100.33) (end 122.174 99.314)
     (stroke (width 0.2) (type default)) (layer "F.Cu"))
+  (gr_line (start 125.73 101.092) (end 123.444 101.092)
+    (stroke (width 0.2) (type default)) (layer "F.Cu"))
   (gr_line (start 139.954 93.98) (end 138.684 93.98)
     (stroke (width 0.2) (type default)) (layer "F.Cu"))
   (gr_line (start 122.174 95.25) (end 121.666 95.25)
     (stroke (width 0.2) (type default)) (layer "F.Cu"))
+  (gr_line (start 125.984 94.742) (end 124.206 94.742)
+    (stroke (width 0.2) (type default)) (layer "F.Cu"))
   (gr_line (start 135.382 109.474) (end 135.382 110.744)
     (stroke (width 0.2) (type default)) (layer "F.Cu"))
   (gr_line (start 124.206 97.282) (end 123.19 97.282)
     (stroke (width 0.2) (type default)) (layer "F.Cu"))
+  (gr_line (start 126.238 103.632) (end 123.444 103.632)
+    (stroke (width 0.2) (type default)) (layer "F.Cu"))
   (gr_line (start 118.11 116.84) (end 118.11 113.284)
     (stroke (width 0.2) (type default)) (layer "F.Cu"))
@@
   (gr_line (start 122.682 98.044) (end 122.682 96.774)
     (stroke (width 0.2) (type default)) (layer "F.Cu"))
+  (gr_line (start 125.984 102.362) (end 123.444 102.362)
+    (stroke (width 0.2) (type default)) (layer "F.Cu"))
   (gr_line (start 138.43 102.616) (end 137.414 102.616)
     (stroke (width 0.2) (type default)) (layer "F.Cu"))
@@
   (gr_line (start 124.206 96.012) (end 123.698 96.012)
     (stroke (width 0.2) (type default)) (layer "F.Cu"))
+  (gr_line (start 125.984 99.822) (end 123.444 99.822)
+    (stroke (width 0.2) (type default)) (layer "F.Cu"))
   (gr_line (start 118.364 106.426) (end 118.364 104.902)
     (stroke (width 0.2) (type default)) (layer "F.Cu"))
@@
   (gr_line (start 135.382 110.998) (end 135.382 112.522)
     (stroke (width 0.2) (type default)) (layer "B.Cu"))
+  (gr_line (start 134.62 111.252) (end 134.62 113.538)
+    (stroke (width 0.2) (type default)) (layer "B.Cu"))
   (gr_line (start 121.285 98.552) (end 121.285 92.837)
