File: Assets/PCB/circle.kicad_pcb (KiCad board)
At the start: 2 copper layers, 40.6 x 40.6 mm, 21 parts, among them j1 R_0805_2012Metric, j10 R_0805_2012Metric, j11 R_0805_2012Metric, j12 R_0805_2012Metric, j13 R_0805_2012Metric, j14 R_0805_2012Metric, j15 R_0805_2012Metric, j2 R_0805_2012Metric, j3 R_0805_2012Metric, j4 R_0805_2012Metric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

Commit message: Update circle.kicad_pcb
Other:
- board text added: "Tactile Sensor PressTip V2.3"
- board text removed: "Tactile Sensor PressTip V2.2"
Changed lines of the file:
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@@
     (effects (font (size 1 1) (thickness 0.1)) (justify left bottom))
   )
-  (gr_text "Tactile Sensor\nPressTip V2.2\n" (at 120.142 86.614) (layer "F.SilkS")
+  (gr_text "Tactile Sensor\nPressTip V2.3\n" (at 120.142 86.614) (layer "F.SilkS")
     (effects (font (size 1 1) (thickness 0.2) bold) (justify left bottom))
   )
